Commit message: Update go2.urdf with mass parameters

File: genesis/assets/urdf/go2/urdf/go2.urdf (robot description, URDF)
Before this commit: robot go2_description, 29 links, 28 joints
Links:
- link base: mass 6.921 -> 10.0

Commit message: change mass in go2_URDF from 10 to 6.921

File: genesis/assets/urdf/go2/urdf/go2.urdf (robot description, URDF)
Before this commit: robot go2_description, 29 links, 28 joints
Links:
- link base: mass 10.0 -> 6.921
