Commit message: Change base mass 11

File: genesis/assets/urdf/go2/urdf/go2_heavy.urdf (robot description, URDF)
Before this commit: robot go2_description, 29 links, 28 joints
Links:
- link base: mass 6.0 -> 11.1

Commit message: Modify go2_heavy.urdf

File: genesis/assets/urdf/go2/urdf/go2_heavy.urdf (robot description, URDF)
Before this commit: robot go2_description, 29 links, 28 joints
Links:
- link base: mass 11.1 -> 15
